Commit message: commit

File: tennis_court/urdf/fledj_bot_description.urdf (robot description, URDF)
Before this commit: robot sam_bot, 8 links, 7 joints
Joints:
- joint pickback_joint: origin xyz=${base_length/2} 0 ${pick_zoff} rpy=0 0 0 -> xyz=${base_length/2+pickback_length/2} 0 ${pick_zoff} rpy=0 0 0
