Commit message: Modif shape robot

File: ws/src/tennis_court/urdf/fledj_bot_description.urdf (robot description, URDF)
Before this commit: robot sam_bot, 7 links, 6 joints
Joints:
- joint base_joint: origin xyz=0.0 0.0 ${-(wheel_radius+wheel_zoff)} rpy=0 0 0 -> xyz=0 0 ${-(wheel_radius+wheel_zoff)} rpy=0 0 0

Commit message: marqueurs visuels pour positionnement

File: ws/src/tennis_court/urdf/fledj_bot_description.urdf (robot description, URDF)
Before this commit: robot sam_bot, 7 links, 6 joints
Joints:
- joint caster_joint: origin xyz=${caster_xoff} 0.0 ${-(base_height/2)} rpy=0 0 0 -> xyz=${caster_xoff} 0.0 ${-base_height/2} rpy=0 0 0

Commit message: correction bugs

File: ws/src/tennis_court/urdf/fledj_bot_description.urdf (robot description, URDF)
Before this commit: robot sam_bot, 7 links, 6 joints
Joints:
- joint caster_joint: origin xyz=${caster_xoff} 0.0 ${-base_height/2} rpy=0 0 0 -> xyz=${caster_xoff} 0.0 ${-(base_height/2)} rpy=0 0 0
